Commit message: feat: AGV 전환 완료 + ESP32-S3 CAN/BLDC 마이그레이션 시작
Phase 1~D (STM32 AGV 전환):
- STM32 EtherCAT→AGV 변환 (main.c 2044→350줄, 레거시 18개 파일 삭제)
- AGV 패킷 프로토콜 0x30~0x34 구현
- ROS2 스택 (Nav2, RTAB-Map, row_follower, obstacle_classifier)
- Phase D: I/O 확장 (io_handler.c, 0x33/0x34 패킷)
- Phase 7: GPS 통합 (U-blox, EKF 융합)
- Web HMI 전면 재작성 (index.html AGV 전용)
- JSON 프로그램 인터프리터 + 편집기 (editor.html)
- systemd 서비스 파일 (agv-nav/ros/slam.service)

Phase E (ESP32-S3 CAN+BLDC 마이그레이션):
- ESP32_CAN_AGV_PLAN.md: 전체 마이그레이션 계획서
- ESP32/agv_firmware: PlatformIO 펌웨어 스켈레톤
  - rs485_slip.cpp: SLIP+CRC16-CCITT (921600 baud)
  - vesc_can.cpp: VESC CAN 드라이버 (500kbps, COMM_SET_RPM)
  - odometry.cpp: ERPM→오도메트리 적분
  - nvs_params.cpp: NVS 파라미터 저장
  - agv_protocol.cpp: 패킷 핸들러 0x30~0x34
  - main.cpp: FreeRTOS 4태스크 구조
- ESP32/vendor/T-CAN485: LILYGO T-CAN485 예제 코드
- 빌드+업로드 확인 완료 (ESP32-D0WDQ6-V3)

Co-Authored-By: Claude Sonnet 4.6 <noreply@anthropic.com>

File: ros2_ws/src/agv_description/urdf/agv.urdf.xacro (robot description, xacro)
@@ -99,4 +99,19 @@
     <axis xyz="0 1 0"/>
   </joint>
+  <!-- ── GPS antenna link (U-blox receiver) ───────────────────────────── -->
+  <!--
+    gps_link: GPS 안테나 위치.
+    navsat_transform_node의 frame_id 와 일치해야 함 (gps_driver_node: frame_id='gps_link').
+    xyz: 로봇 중심 기준 오프셋 (현장 실측 후 수정)
+      x=0.0  — 전후 중앙
+      y=0.0  — 좌우 중앙
+      z=0.35 — base_height(0.20) + 여유 0.15m (안테나 상단)
+  -->
+  <link name="gps_link"/>
+  <joint name="gps_joint" type="fixed">
+    <parent link="base_link"/>
+    <child  link="gps_link"/>
+    <origin xyz="0.0 0.0 0.35" rpy="0 0 0"/>
+  </joint>
   <!-- ── Camera link (Intel RealSense D435/D455) ───────────────────────── -->
   <!--
